Commit message: Changed model files to support urdf for pybullet.

File: urdf/digit_model.urdf (robot description, URDF)
Before this commit: robot digit, 29 links, 28 joints
Links:
- link left_elbow: geometry collision mesh filename=package://urdf/arm-L4.obj; visual mesh filename=package://urdf/arm-L4.obj
- link left_hip_pitch: geometry collision mesh filename=package://urdf/hip-pitch.obj; visual mesh filename=package://urdf/hip-pitch.obj
- link left_hip_roll: geometry collision mesh filename=package://urdf/hip-yaw-housing.obj; visual mesh filename=package://urdf/hip-yaw-housing.obj
- link left_hip_yaw: geometry collision mesh filename=package://urdf/hip-pitch-housing.obj; visual mesh filename=package://urdf/hip-pitch-housing.obj
- link left_knee: geometry collision mesh filename=package://urdf/knee.obj; visual mesh filename=package://urdf/knee.obj
- link left_shin: geometry collision mesh filename=package://urdf/shin.obj; visual mesh filename=package://urdf/shin.obj
- link left_shoulder_cap: geometry collision mesh filename=package://urdf/shoulder-roll-housing.obj; visual mesh filename=package://urdf/shoulder-roll-housing.obj
- link left_shoulder_pitch: geometry collision mesh filename=package://urdf/arm-L2.obj; visual mesh filename=package://urdf/arm-L2.obj
- link left_shoulder_roll: geometry collision mesh filename=package://urdf/arm-L1.obj; visual mesh filename=package://urdf/arm-L1.obj
- link left_shoulder_yaw: geometry collision mesh filename=package://urdf/arm-L3.obj; visual mesh filename=package://urdf/arm-L3.obj
- link left_tarsus: geometry collision mesh filename=package://urdf/tarsus.obj; visual mesh filename=package://urdf/tarsus.obj
- link left_toe_pitch: geometry collision mesh filename=package://urdf/toe-pitch.obj; visual mesh filename=package://urdf/toe-pitch.obj
- link left_toe_roll: geometry collision mesh filename=package://urdf/toe-roll.obj; visual mesh filename=package://urdf/toe-roll.obj
- link left_waist_cap: geometry collision mesh filename=package://urdf/shoulder-roll-housing.obj; visual mesh filename=package://urdf/shoulder-roll-housing.obj
- link right_elbow: geometry collision mesh filename=package://urdf/arm-L4.obj scale=1 -1 1; visual mesh filename=package://urdf/arm-L4.obj scale=1 -1 1
- link right_hip_pitch: geometry collision mesh filename=package://urdf/hip-pitch.obj scale=1 -1 1; visual mesh filename=package://urdf/hip-pitch.obj scale=1 -1 1
- link right_hip_roll: geometry collision mesh filename=package://urdf/hip-yaw-housing.obj scale=1 -1 1; visual mesh filename=package://urdf/hip-yaw-housing.obj scale=1 -1 1
- link right_hip_yaw: geometry collision mesh filename=package://urdf/hip-pitch-housing.obj scale=1 -1 1; visual mesh filename=package://urdf/hip-pitch-housing.obj scale=1 -1 1
- link right_knee: geometry collision mesh filename=package://urdf/knee.obj scale=1 -1 1; visual mesh filename=package://urdf/knee.obj scale=1 -1 1
- link right_shin: geometry collision mesh filename=package://urdf/shin.obj scale=1 -1 1; visual mesh filename=package://urdf/shin.obj scale=1 -1 1
- link right_shoulder_cap: geometry collision mesh filename=package://urdf/shoulder-roll-housing.obj scale=1 -1 1; visual mesh filename=package://urdf/shoulder-roll-housing.obj scale=1 -1 1
- link right_shoulder_pitch: geometry collision mesh filename=package://urdf/arm-L2.obj scale=1 -1 1; visual mesh filename=package://urdf/arm-L2.obj scale=1 -1 1
- link right_shoulder_roll: geometry collision mesh filename=package://urdf/arm-L1.obj scale=1 -1 1; visual mesh filename=package://urdf/arm-L1.obj scale=1 -1 1
- link right_shoulder_yaw: geometry collision mesh filename=package://urdf/arm-L3.obj scale=1 -1 1; visual mesh filename=package://urdf/arm-L3.obj scale=1 -1 1
- link right_tarsus: geometry collision mesh filename=package://urdf/tarsus.obj scale=1 -1 1; visual mesh filename=package://urdf/tarsus.obj scale=1 -1 1
- link right_toe_pitch: geometry collision mesh filename=package://urdf/toe-pitch.obj scale=1 -1 1; visual mesh filename=package://urdf/toe-pitch.obj scale=1 -1 1
- link right_toe_roll: geometry collision mesh filename=package://urdf/toe-roll.obj scale=1 -1 1; visual mesh filename=package://urdf/toe-roll.obj scale=1 -1 1
- link right_waist_cap: geometry collision mesh filename=package://urdf/shoulder-roll-housing.obj scale=1 -1 1; visual mesh filename=package://urdf/shoulder-roll-housing.obj scale=1 -1 1
- link torso: geometry collision mesh filename=package://urdf/torso.obj; visual mesh filename=package://urdf/torso.obj
Joints:
- removed joint left-elbow
- removed joint left-hip-pitch
- removed joint left-hip-roll
- removed joint left-hip-yaw
- removed joint left-knee
- removed joint left-shin
- removed joint left-shoulder-pitch
- removed joint left-shoulder-roll
- removed joint left-shoulder-yaw
- removed joint left-tarsus
- removed joint left-toe-pitch
- removed joint left-toe-roll
- removed joint right-elbow
- removed joint right-hip-pitch
- removed joint right-hip-roll
- removed joint right-hip-yaw
- removed joint right-knee
- removed joint right-shin
- removed joint right-shoulder-pitch
- removed joint right-shoulder-roll
- removed joint right-shoulder-yaw
- removed joint right-tarsus
- removed joint right-toe-pitch
- removed joint right-toe-roll
- added joint elbow_joint_left: type continuous, parent left_shoulder_yaw, child left_elbow, origin xyz=0 -0.0385 0.185 rpy=1.57079632679 -0.3926991 0, axis 0 0 1, limit lower=-1.3526 upper=1.3526 effort=1.4 velocity=12.5
- added joint elbow_joint_right: type continuous, parent right_shoulder_yaw, child right_elbow, origin xyz=0 0.0385 0.185 rpy=-1.57079632679 -0.3926991 0, axis 0 0 1, limit lower=-1.3526 upper=1.3526 effort=1.4 velocity=12.5
- added joint hip_abduction_left: type continuous, parent torso, child left_hip_roll, origin xyz=-0.001 0.091 0 rpy=1.57079632679 -1.1955506 -1.57079632679, axis 0 0 1, limit lower=-1.0472 upper=1.0472 effort=1.4 velocity=12.15
- added joint hip_abduction_right: type continuous, parent torso, child right_hip_roll, origin xyz=-0.001 -0.091 0 rpy=-1.57079632679 -1.1955506 1.57079632679, axis 0 0 1, limit lower=-1.0472 upper=1.0472 effort=1.4 velocity=12.15
- added joint hip_flexion_left: type continuous, parent left_hip_yaw, child left_hip_pitch, origin xyz=0 0.004 0.068 rpy=-1.57079632679 -0.785398163397 3.14159265359, axis 0 0 -1, limit lower=-1.0472 upper=1.57079632679 effort=12.5 velocity=8.5
- added joint hip_flexion_right: type continuous, parent right_hip_yaw, child right_hip_pitch, origin xyz=0 -0.004 0.068 rpy=1.57079632679 -0.785398163397 -3.14159265359, axis 0 0 -1, limit lower=-1.57079632679 upper=1.0472 effort=12.5 velocity=8.5
- added joint hip_rotation_left: type continuous, parent left_hip_roll, child left_hip_yaw, origin xyz=-0.0505 0 0.044 rpy=0 -1.57079632679 0, axis 0 0 1, limit lower=-0.698132 upper=0.698132 effort=1.4 velocity=12.15
- added joint hip_rotation_right: type continuous, parent right_hip_roll, child right_hip_yaw, origin xyz=-0.0505 0 0.044 rpy=0 -1.57079632679 0, axis 0 0 1, limit lower=-0.698132 upper=0.698132 effort=1.4 velocity=12.15
- added joint knee_joint_left: type continuous, parent left_hip_pitch, child left_knee, origin xyz=0.12 0 0.0045 rpy=0 0 -1.57079632679, axis 0 0 1, limit lower=-1.2392 upper=0.8727 effort=12.5 velocity=8.5085
- added joint knee_joint_right: type continuous, parent right_hip_pitch, child right_knee, origin xyz=0.12 0 0.0045 rpy=0 0 1.57079632679, axis 0 0 1, limit lower=-0.8727 upper=1.2392 effort=12.5 velocity=8.5085
- added joint knee_to_shin_left: type fixed, parent left_knee, child left_shin, origin xyz=0.060677 0.047406 0 rpy=0 0 0, axis 0 0 1, limit lower=-0.35 upper=0.35 effort=0 velocity=10
- added joint knee_to_shin_right: type fixed, parent right_knee, child right_shin, origin xyz=0.060677 -0.047406 0 rpy=0 0 0, axis 0 0 1, limit lower=-0.35 upper=0.35 effort=0 velocity=10
- added joint shin_to_tarsus_left: type continuous, parent left_shin, child left_tarsus, origin xyz=0.434759 0.02 0 rpy=0 0 1.7976891, axis 0 0 1, limit lower=-0.8779 upper=1.2497 effort=0 velocity=20
- added joint shin_to_tarsus_right: type continuous, parent right_shin, child right_tarsus, origin xyz=0.434759 -0.02 0 rpy=0 0 -1.7976891, axis 0 0 1, limit lower=-1.2497 upper=0.8779 effort=0 velocity=20
- added joint shoulder_pitch_joint_left: type continuous, parent left_shoulder_roll, child left_shoulder_pitch, origin xyz=-0.00317 -0.011055 0.0555 rpy=1.57079632679 0.785398163397 -0.2792527, axis 0 0 -1, limit lower=-2.5307 upper=2.5307 effort=1.4 velocity=12.5
- added joint shoulder_pitch_joint_right: type continuous, parent right_shoulder_roll, child right_shoulder_pitch, origin xyz=-0.00317 0.011055 0.0555 rpy=-1.57079632679 0.785398163397 0.2792527, axis 0 0 -1, limit lower=-2.5307 upper=2.5307 effort=1.4 velocity=12.5
- added joint shoulder_roll_joint_left: type continuous, parent torso, child left_shoulder_roll, origin xyz=-0.001 0.12 0.4 rpy=-1.57079632679 -1.3962633 1.57079632679, axis 0 0 1, limit lower=-1.309 upper=1.309 effort=1.4 velocity=12.5
- added joint shoulder_roll_joint_right: type continuous, parent torso, child right_shoulder_roll, origin xyz=-0.001 -0.12 0.4 rpy=1.57079632679 -1.3962633 -1.57079632679, axis 0 0 1, limit lower=-1.309 upper=1.309 effort=1.4 velocity=12.5
- added joint shoulder_yaw_joint_left: type continuous, parent left_shoulder_pitch, child left_shoulder_yaw, origin xyz=0 -0.165 -0.1 rpy=1.57079632679 0 0, axis 0 0 1, limit lower=-1.7453 upper=1.7453 effort=1.4 velocity=10
- added joint shoulder_yaw_joint_right: type continuous, parent right_shoulder_pitch, child right_shoulder_yaw, origin xyz=0 0.165 -0.1 rpy=-1.57079632679 0 0, axis 0 0 1, limit lower=-1.7453 upper=1.7453 effort=1.4 velocity=10
- added joint toe_pitch_joint_left: type continuous, parent left_tarsus, child left_toe_pitch, origin xyz=0.408 -0.04 0 rpy=0 0 1.1956, axis 0 0 1, limit lower=-0.785398163397 upper=0.785398163397 effort=0.9 velocity=11.5
- added joint toe_pitch_joint_right: type continuous, parent right_tarsus, child right_toe_pitch, origin xyz=0.408 0.04 0 rpy=0 0 -1.1956, axis 0 0 1, limit lower=-0.785398163397 upper=0.785398163397 effort=0.9 velocity=11.5
- added joint toe_roll_joint_left: type continuous, parent left_toe_pitch, child left_toe_roll, origin xyz=0 0 0 rpy=0 1.57079632679 0, axis 0 0 1, limit lower=-0.6109 upper=0.6109 effort=0.9 velocity=11.5
- added joint toe_roll_joint_right: type continuous, parent right_toe_pitch, child right_toe_roll, origin xyz=0 0 0 rpy=0 1.57079632679 0, axis 0 0 1, limit lower=-0.6109 upper=0.6109 effort=0.9 velocity=11.5
